Commit message: fix: move mpo_700 IMU up to z=0.2 to avoid ground clipping

File: robots/mpo_700/urdf/imu.xacro (robot description, xacro)
@@ -3,5 +3,5 @@
     <joint name="imu_sensor_joint" type="fixed">
         <axis xyz="0 0 1" />
-        <origin xyz="0 0 0" rpy="0 0 0"/>
+        <origin xyz="0 0 0.2" rpy="0 0 0"/>
         <parent link="base_link"/>
         <child link="imu_sensor_link"/>
