Commit message: add customized sensors

File: robots/mpo_700/mpo_700.urdf.xacro (robot description, xacro)
@@ -49,3 +49,21 @@
       <!-- Sick S300 - Comment/Uncomment if required -->
       <!-- <xacro:include filename="$(find neo_simulation2)/robots/mpo_700/xacros/sick_S300.xacro" /> -->
+    <xacro:include filename="$(find neo_simulation2)/robots/mpo_700/urdf/inertial_macros.xacro"/>
+    <xacro:include filename="$(find neo_simulation2)/robots/mpo_700/urdf/lidar.xacro" />
+    <xacro:include filename="$(find neo_simulation2)/robots/mpo_700/urdf/depth_camera.xacro" />
+    <xacro:include filename="$(find neo_simulation2)/robots/mpo_700/urdf/ultrasonic_sensor.xacro" />
+    <!-- origin is the position between chassis and realsense d435i -->
+    <!-- <xacro:include filename="_d435i.urdf.xacro"/>
+    <xacro:sensor_d435i parent="chassis" name="camera" topics_ns="camera">
+        <origin xyz="0.35 0.0 0.13" rpy="0.0 0.0 0.0"/>
+    </xacro:sensor_d435i> -->
+    <!-- Test!! -->
+    <!-- <link name="base_link" /> -->
+    <!-- <xacro:include filename="depth_camera.xacro" /> -->
+    <!-- <xacro:include filename="camera.xacro"/> -->
+<!--
+    <xacro:include filename="_d435i.urdf.xacro"/>
+    <xacro:sensor_d435i parent="base_link" name="camera" topics_ns="camera">
+        <origin xyz="0.0 0.0 0.13" rpy="0.0 0.0 0.0"/>
+    </xacro:sensor_d435i> -->
 </robot>

File: robots/mpo_700/urdf/mpo_700_body.urdf.xacro (robot description, xacro)
@@ -32,5 +32,5 @@
     <joint name="lidar_1_joint" type="fixed">
         <axis xyz="0 1 0"/>
-        <origin rpy="3.14 0 0.79" xyz="0.338 0.288 0.223"/>
+        <origin rpy="0 0 0" xyz="0.1 0.1 1"/>
         <parent link="base_link"/>
         <child link="lidar_1_link"/>
@@ -41,29 +41,4 @@
             <origin rpy="0 0 0" xyz="0 0 0"/>
             <inertia ixx="0.11042056" ixy="0.0" ixz="0.0" iyy="0.11042056" iyz="0.0" izz="0.11042056"/>
-        </inertial>
-        <visual>
-            <origin rpy="-1.57 0 3.14" xyz="0 0 -0.12"/>
-            <geometry>
-                <mesh filename="package://neo_simulation2/components/meshes/SICK-S300.dae" scale="0.001 0.001 0.001"/>
-            </geometry>
-        </visual>
-        <collision>
-            <origin rpy="-1.57 0 3.14" xyz="0 0 -0.12"/>
-            <geometry>
-                <mesh filename="package://neo_simulation2/components/meshes/SICK-S300.dae" scale="0.001 0.001 0.001"/>
-            </geometry>
-        </collision>
-    </link>
-    <joint name="lidar_2_joint" type="fixed">
-        <axis xyz="0 1 0"/>
-        <origin rpy="3.14 0 3.93" xyz="-0.338 -0.288 0.223"/>
-        <parent link="base_link"/>
-        <child link="lidar_2_link"/>
-    </joint>
-    <link name="lidar_2_link" type="laser">
-        <inertial>
-            <mass value="0.001"/>
-            <origin rpy="0 0 0" xyz="0 0 0"/>
-            <inertia ixx="0.0001" ixy="0" ixz="0" iyy="0.000001" iyz="0" izz="0.0001"/>
         </inertial>
         <visual>

File: robots/mpo_700/urdf/mpo_700_gazebo.urdf.xacro (robot description, xacro)
@@ -6,8 +6,7 @@
     <xacro:include filename="$(find neo_simulation2)/robots/mpo_700/urdf/macro/gazebo_mpo_700_wheel_macro.xacro" />
     <!-- Properties -->
-    <xacro:property name="lidar_1_update_rate" value="40" />
-    <xacro:property name="lidar_2_update_rate" value="40" />
-    <xacro:property name="controller_update_rate" value="100" />
-    <xacro:property name="odom_update_rate" value="100" />
+    <xacro:property name="lidar_1_update_rate" value="10" />
+    <xacro:property name="controller_update_rate" value="10" />
+    <xacro:property name="odom_update_rate" value="10" />
     <!--Object Controller-->
     <xacro:gazebo_object_controller
@@ -23,26 +22,12 @@
         link_name="lidar_1_link"
         update_rate="${lidar_1_update_rate}"
-        min_range="0.10"
-        max_range="30.0"
-        horizontal_samples="720"
-        min_angle="-1.48"
-        max_angle="1.48"
+        min_range="0.1"
+        max_range="10.0"
+        horizontal_samples="360"
+        min_angle="-3.14"
+        max_angle="3.14"
         noise_mean="0.0"
-        noise_stddev="0.01"
+        noise_stddev="0.02"
         topic_name="scan"
-        visualize="false"
-    />
-    <xacro:gazebo_lidar_sensor
-        sensor_name="lidar_2_sensor"
-        link_name="lidar_2_link"
-        update_rate="${lidar_2_update_rate}"
-        min_range="0.10"
-        max_range="30.0"
-        horizontal_samples="720"
-        min_angle="-1.48"
-        max_angle="1.48"
-        noise_mean="0.0"
-        noise_stddev="0.01"
-        topic_name="scan2"
         visualize="false"
     />

Commit message: Add 9-DOF IMU to MPO-700 at base center
- Fix imu.xacro to use base_link parent and place at (0,0,0)
- Include imu.xacro in mpo_700.urdf.xacro

File: robots/mpo_700/mpo_700.urdf.xacro (robot description, xacro)
@@ -53,4 +53,5 @@
     <xacro:include filename="$(find neo_simulation2)/robots/mpo_700/urdf/depth_camera.xacro" />
     <xacro:include filename="$(find neo_simulation2)/robots/mpo_700/urdf/ultrasonic_sensor.xacro" />
+    <xacro:include filename="$(find neo_simulation2)/robots/mpo_700/urdf/imu.xacro" />
     <!-- origin is the position between chassis and realsense d435i -->
     <!-- <xacro:include filename="_d435i.urdf.xacro"/>

File: robots/mpo_700/urdf/imu.xacro (robot description, xacro)
@@ -3,6 +3,6 @@
     <joint name="imu_sensor_joint" type="fixed">
         <axis xyz="0 0 1" />
-        <origin xyz="${chassis_length} 0 ${chassis_height/2}" rpy="0 0 0"/>
-        <parent link="chassis"/>
+        <origin xyz="0 0 0" rpy="0 0 0"/>
+        <parent link="base_link"/>
         <child link="imu_sensor_link"/>
     </joint>
@@ -30,5 +30,5 @@
         <sensor name='imu_sensor' type='imu'>
             <always_on>1</always_on>
-            <update_rate>1000</update_rate>
+            <update_rate>100</update_rate>
             <visualize>1</visualize>
             <topic>__default_topic__</topic>
@@ -36,9 +36,8 @@
                 <ros>
                     <!-- Will publish to /imu/data -->
-                    <namespace>/camera</namespace>
-                    <remapping>~/out:=imu</remapping>
+                    <remapping>~/out:=imu/data</remapping>
                 </ros>
-                <bodyName>imu_sensor_link</bodyName>
-                <updateRateHZ>10.0</updateRateHZ>
+                <frameName>imu_sensor_link</frameName>
+                <updateRateHZ>100.0</updateRateHZ>
                 <gaussianNoise>0.0</gaussianNoise>
                 <xyzOffset>0 0 0</xyzOffset>

Commit message: feat(mpo_700): add 360° 2D lidar at 1.0m (/scan_all) and disable 3D lidar + RGBD camera
Changes:
- Add lidar_all_link at 1.0m height with cylindrical visual/collision
- Add gazebo_lidar_sensor publishing /scan_all:
  - 1125 samples @ 0.32° angular resolution (360° coverage)
  - 0.3m min range, 30m max range
  - ±1cm precision (noise stddev 0.0033)
  - visualize=false
- Disable Velodyne 3D lidar (lidar.xacro) and RGBD camera (depth_camera.xacro)
- Update existing lidar_1_sensor to 1125 samples for consistency

File: robots/mpo_700/mpo_700.urdf.xacro (robot description, xacro)
@@ -50,6 +50,8 @@
       <!-- <xacro:include filename="$(find neo_simulation2)/robots/mpo_700/xacros/sick_S300.xacro" /> -->
     <xacro:include filename="$(find neo_simulation2)/robots/mpo_700/urdf/inertial_macros.xacro"/>
-    <xacro:include filename="$(find neo_simulation2)/robots/mpo_700/urdf/lidar.xacro" />
-    <xacro:include filename="$(find neo_simulation2)/robots/mpo_700/urdf/depth_camera.xacro" />
+    <!-- 3D LIDAR DISABLED -->
+    <!-- <xacro:include filename="$(find neo_simulation2)/robots/mpo_700/urdf/lidar.xacro" /> -->
+    <!-- RGBD CAMERA DISABLED -->
+    <!-- <xacro:include filename="$(find neo_simulation2)/robots/mpo_700/urdf/depth_camera.xacro" /> -->
     <xacro:include filename="$(find neo_simulation2)/robots/mpo_700/urdf/ultrasonic_sensor.xacro" />
     <xacro:include filename="$(find neo_simulation2)/robots/mpo_700/urdf/imu.xacro" />

File: robots/mpo_700/urdf/mpo_700_body.urdf.xacro (robot description, xacro)
@@ -52,4 +52,31 @@
             <geometry>
                 <mesh filename="package://neo_simulation2/components/meshes/SICK-S300.dae" scale="0.001 0.001 0.001"/>
+            </geometry>
+        </collision>
+    </link>
+    <!-- 360-degree 2D Lidar at 1.0m height -->
+    <joint name="lidar_all_joint" type="fixed">
+        <axis xyz="0 1 0"/>
+        <origin rpy="0 0 0" xyz="0 0 1.0"/>
+        <parent link="base_link"/>
+        <child link="lidar_all_link"/>
+    </joint>
+    <link name="lidar_all_link" type="laser">
+        <inertial>
+            <mass value="0.5"/>
+            <origin rpy="0 0 0" xyz="0 0 0"/>
+            <inertia ixx="0.01" ixy="0.0" ixz="0.0" iyy="0.01" iyz="0.0" izz="0.01"/>
+        </inertial>
+        <visual>
+            <origin rpy="0 0 0" xyz="0 0 0"/>
+            <geometry>
+                <cylinder radius="0.04" length="0.06"/>
+            </geometry>
+            <material name="red"/>
+        </visual>
+        <collision>
+            <origin rpy="0 0 0" xyz="0 0 0"/>
+            <geometry>
+                <cylinder radius="0.04" length="0.06"/>
             </geometry>
         </collision>

File: robots/mpo_700/urdf/mpo_700_gazebo.urdf.xacro (robot description, xacro)
@@ -24,5 +24,5 @@
         min_range="0.5"
         max_range="10.0"
-        horizontal_samples="360"
+        horizontal_samples="1125"
         min_angle="-3.14"
         max_angle="3.14"
@@ -30,4 +30,19 @@
         noise_stddev="0.02"
         topic_name="scan"
+        visualize="false"
+    />
+    <!-- 360-degree 2D Lidar at 1.0m height -->
+    <xacro:gazebo_lidar_sensor
+        sensor_name="lidar_all_sensor"
+        link_name="lidar_all_link"
+        update_rate="10"
+        min_range="0.3"
+        max_range="30.0"
+        horizontal_samples="1125"
+        min_angle="-3.14159"
+        max_angle="3.14159"
+        noise_mean="0.0"
+        noise_stddev="0.0033"
+        topic_name="scan_all"
         visualize="false"
     />
